File: atmega328-adapter/atmega328-adapter.kicad_sch (KiCad schematic)
At the start: 1 part, among them U1 ATmega168A-A

Commit message: updated adapter
Parts:
- added J1, J2: Conn_01x14, Connector_PinHeader_2.54mm:PinHeader_1x14_P2.54mm_Vertical, symbol Connector_Generic:Conn_01x14
Connections:
- net +5V: now also J1.7 (Pin_7), J2.8 (Pin_8), J2.9 (Pin_9)
- net CS: now also J2.13 (Pin_13)
- net GND: now also J1.8 (Pin_8), J2.7 (Pin_7)
- net MISO: now also J2.11 (Pin_11)
- net MOSI: now also J2.12 (Pin_12)
- net PB0: now also J1.14 (Pin_14)
- net PB1: now also J2.14 (Pin_14)
- net PB5: now also J2.10 (Pin_10)
- net PC0: now also J2.6 (Pin_6)
- net PC1: now also J2.5 (Pin_5)
- net PC2: now also J2.4 (Pin_4)
- net PC3: now also J2.3 (Pin_3)
- net PC4: now also J2.2 (Pin_2)
- net PC5: now also J2.1 (Pin_1)
- net PD0: now also J1.2 (Pin_2)
- net PD1: now also J1.3 (Pin_3)
- net PD2: now also J1.4 (Pin_4)
- net PD3: now also J1.5 (Pin_5)
- net PD4: now also J1.6 (Pin_6)
- net PD5: now also J1.11 (Pin_11)
- net PD6: now also J1.12 (Pin_12)
- net PD7: now also J1.13 (Pin_13)
- net RESET: now also J1.1 (Pin_1)
- net XTAL1: now also J1.9 (Pin_9)
- net XTAL2: now also J1.10 (Pin_10)
